File: Hardware/All In One PCB/Voltmeter PCB RTC ESP_v3.brd (EAGLE design)
At the start: 36.8 x 36.8 mm, 27 parts, among them U3 INA226AIDGSR

Commit message: PCB Update
Parts:
- moved CR1220 1.27 mm to (30.7, 17.8)
- moved GND 1.27 mm to (29.2, 31.9)
- moved R2 1.27 mm to (32.8, 17.3)
- moved R5 1.27 mm to (32.8, 17.3)
- moved SRC- 1.27 mm to (29.2, 5.08)
- moved IN 1.27 mm to (35.7, 2.54)
- moved OUT 1.27 mm to (35.7, 31.9)
Routing:
- net IN+: track 96.0 -> 105.6 mm, vias 25 -> 26
- net IN-: track 42.3 -> 47.6 mm, vias 22 -> 23
- net S_GND: track 38.7 -> 41.3 mm
- net RTC_BAT: track 48.6 -> 49.4 mm
- net GND: track 22.2 -> 22.8 mm
Other:
- board size 36.8 x 36.8 mm -> 38.1 x 36.8 mm
